File: pico-ethernet.kicad_sch (KiCad schematic)
At the start: 29 parts, among them J1 Conn_01x20_Pin, J2 Conn_01x02, J3 VR05S05, J4 SI-52003-F, J5 Conn_01x02, J6 Conn_01x02_Pin, U1 ENC28J60x-SS, Y1 25MHz

Commit message: redux 1?
Parts:
- removed J2: Conn_01x02, Connector_JST:JST_SH_SM02B-SRSS-TB_1x02-1MP_P1.00mm_Horizontal, symbol Connector_Generic:Conn_01x02
- J2: renamed from J6; footprint Connector_PinSocket_2.54mm:PinSocket_1x02_P2.54mm_Vertical -> Connector_PinSocket_2.54mm:PinSocket_1x04_P2.54mm_Vertical; symbol Connector:Conn_01x02_Pin -> Connector:Conn_01x04_Pin
- J5: footprint Connector_JST:JST_SH_SM02B-SRSS-TB_1x02-1MP_P1.00mm_Horizontal -> TerminalBlock_Phoenix:TerminalBlock_Phoenix_MPT-0,5-4-2.54_1x04_P2.54mm_Horizontal; symbol Connector_Generic:Conn_01x02 -> Connector:Screw_Terminal_01x04
Connections:
- net GND: now also J2.3 (Pin_3), J5.1 (Pin_1); no longer J5.2 (Pin_2)
- net at J2.2 (Pin_2): now also J5.3 (Pin_3)
- net at R6.1: now also U1.27 (LEDA); no longer U1.26 (LEDB)
- net at J2.1 (Pin_1): now also J5.4 (Pin_4); no longer J5.1 (Pin_1)
- net at R7.1: now also U1.26 (LEDB); no longer U1.27 (LEDA)
- new net: J2.4 (Pin_4), J5.2 (Pin_2)
